Commit message: fix(gazebo): stop degenerate contacts from turning joint state into NaN
Every arm link's collision box ends exactly where the next one
starts (shoulder ends at z=0.5, arm starts at z=0.5, ...) and their
x/y footprints fully overlap. base_link's bottom face likewise lands
exactly on the z=0 ground plane. These zero-penetration, face-to-face
contacts are degenerate for ODE's constraint solver: it can resolve
them to NaN, which shows up as

  * every joint reporting velocity = NaN, effort = NaN
  * the affected links' poses going NaN, so Gazebo silently stops
    rendering them -- "only the base is left"

Disable collision between adjacent links (they should never collide
with each other anyway, and it also stops the contact solver from
fighting the joint PIDs), and spawn the robot 1 cm above the ground so
the base lands instead of being exactly coplanar with it.

Also print the real per-link pose from Gazebo 10 s after spawn, so the
state of the model can be inspected without a screenshot.

Co-Authored-By: deepseek <deepseek@anthropic.com>

File: ros2_ws/src/my_robot_description/urdf/my_robot.gazebo.ros2_control.xacro (robot description, xacro)
@@ -75,3 +75,42 @@
     </plugin>
   </gazebo>
+  <!-- 关闭相邻连杆之间的碰撞。
+       本 URDF 里每一段的碰撞盒都"正好贴着"下一段（面面共面，X/Y 完全重叠），
+       这种零穿透的退化接触会让 ODE 的约束求解器解出 NaN：
+       关节 velocity/effort 变成 NaN，连杆位姿变成 NaN，
+       Gazebo 渲染时 NaN 位姿的连杆直接不显示 —— 表现就是"只剩底座，机械臂不见了"。
+       机器人自身的相邻连杆本来就不该互相碰撞，关掉同时也避免
+       碰撞求解器跟关节 PID 抢力矩（机械臂会抖、会飞）。 -->
+  <gazebo>
+    <joint name="joint1">
+      <parent>base_link</parent>
+      <child>shoulder_link</child>
+      <disable_collide>true</disable_collide>
+    </joint>
+    <joint name="joint2">
+      <parent>shoulder_link</parent>
+      <child>arm_link</child>
+      <disable_collide>true</disable_collide>
+    </joint>
+    <joint name="joint3">
+      <parent>arm_link</parent>
+      <child>elbow_link</child>
+      <disable_collide>true</disable_collide>
+    </joint>
+    <joint name="joint4">
+      <parent>elbow_link</parent>
+      <child>forearm_link</child>
+      <disable_collide>true</disable_collide>
+    </joint>
+    <joint name="joint5">
+      <parent>forearm_link</parent>
+      <child>wrist_link</child>
+      <disable_collide>true</disable_collide>
+    </joint>
+    <joint name="joint6">
+      <parent>wrist_link</parent>
+      <child>hand_link</child>
+      <disable_collide>true</disable_collide>
+    </joint>
+  </gazebo>
 </robot>
