Commit message: feat(description): add inertial properties for Gazebo physics
Add mass and inertia tensors to every link in arm.xacro and
gripper.xacro so my_robot can be simulated in Gazebo's physics
engine. base_link is made heavier (5 kg) for stability.

Co-Authored-By: deepseek <deepseek@users.noreply.github.com>

File: ros2_ws/src/my_robot_description/urdf/arm.xacro (robot description, xacro)
@@ -16,4 +16,9 @@
             <origin xyz="0 0 0.05" rpy="0 0 0"/>
         </collision>
+        <inertial>
+            <origin xyz="0 0 0.05" rpy="0 0 0"/>
+            <mass value="5.0"/>
+            <inertia ixx="0.070833" ixy="0" ixz="0" iyy="0.070833" iyz="0" izz="0.133333"/>
+        </inertial>
     </link>
     <!-- shoulder_link: cylinder length 0.5 radius 0.1 -->
@@ -32,4 +37,9 @@
             <origin xyz="0 0 0.25" rpy="0 0 0"/>
         </collision>
+        <inertial>
+            <origin xyz="0 0 0.25" rpy="0 0 0"/>
+            <mass value="0.5"/>
+            <inertia ixx="0.011667" ixy="0" ixz="0" iyy="0.011667" iyz="0" izz="0.0025"/>
+        </inertial>
     </link>
     <!-- arm_link: cylinder length 0.6 radius 0.05 -->
@@ -49,4 +59,9 @@
             <origin xyz="0 0 0.3" rpy="0 0 0"/>
         </collision>
+        <inertial>
+            <origin xyz="0 0 0.3" rpy="0 0 0"/>
+            <mass value="0.3"/>
+            <inertia ixx="0.009188" ixy="0" ixz="0" iyy="0.009188" iyz="0" izz="0.000375"/>
+        </inertial>
     </link>
     <!-- elbow_link: cylinder length 0.1 radius 0.05 -->
@@ -65,4 +80,9 @@
             <origin xyz="0 0 0.05" rpy="0 0 0"/>
         </collision>
+        <inertial>
+            <origin xyz="0 0 0.05" rpy="0 0 0"/>
+            <mass value="0.1"/>
+            <inertia ixx="0.000146" ixy="0" ixz="0" iyy="0.000146" iyz="0" izz="0.000125"/>
+        </inertial>
     </link>
     <!-- forearm_link: cylinder length 0.5 radius 0.05 -->
@@ -82,4 +102,9 @@
             <origin xyz="0 0 0.25" rpy="0 0 0"/>
         </collision>
+        <inertial>
+            <origin xyz="0 0 0.25" rpy="0 0 0"/>
+            <mass value="0.25"/>
+            <inertia ixx="0.005365" ixy="0" ixz="0" iyy="0.005365" iyz="0" izz="0.000313"/>
+        </inertial>
     </link>
     <!-- wrist_link: box size 0.1 0.1 0.05 -->
@@ -98,4 +123,9 @@
             <origin xyz="0 0 0.025" rpy="0 0 0"/>
         </collision>
+        <inertial>
+            <origin xyz="0 0 0.025" rpy="0 0 0"/>
+            <mass value="0.1"/>
+            <inertia ixx="0.000104" ixy="0" ixz="0" iyy="0.000104" iyz="0" izz="0.000167"/>
+        </inertial>
     </link>
     <!-- hand_link: box size 0.1 0.1 0.02 -->
@@ -114,7 +144,18 @@
             <origin xyz="0 0 0.01" rpy="0 0 0"/>
         </collision>
+        <inertial>
+            <origin xyz="0 0 0.01" rpy="0 0 0"/>
+            <mass value="0.05"/>
+            <inertia ixx="0.000043" ixy="0" ixz="0" iyy="0.000043" iyz="0" izz="0.000083"/>
+        </inertial>
     </link>
     <!-- tool_link: no visual -->
-    <link name="tool_link"/>
+    <link name="tool_link">
+        <inertial>
+            <origin xyz="0 0 0" rpy="0 0 0"/>
+            <mass value="0.01"/>
+            <inertia ixx="0.000001" ixy="0" ixz="0" iyy="0.000001" iyz="0" izz="0.000001"/>
+        </inertial>
+    </link>
     <!-- joint1: revolute, axis z, min -3.14, max 3.14 -->
     <joint name="joint1" type="revolute">

File: ros2_ws/src/my_robot_description/urdf/gripper.xacro (robot description, xacro)
@@ -16,4 +16,9 @@
       <origin xyz="0 0 0.01" rpy="0 0 0"/>
     </collision>
+    <inertial>
+      <origin xyz="0 0 0.01" rpy="0 0 0"/>
+      <mass value="0.05"/>
+      <inertia ixx="0.000017" ixy="0" ixz="0" iyy="0.000168" iyz="0" izz="0.000182"/>
+    </inertial>
   </link>
   <!-- 左夹爪手指 -->
@@ -32,4 +37,9 @@
       <origin xyz="0 0 0.04" rpy="0 0 0"/>
     </collision>
+    <inertial>
+      <origin xyz="0 0 0.04" rpy="0 0 0"/>
+      <mass value="0.02"/>
+      <inertia ixx="0.000017" ixy="0" ixz="0" iyy="0.000011" iyz="0" izz="0.000007"/>
+    </inertial>
   </link>
   <!-- 右夹爪手指 -->
@@ -48,4 +58,9 @@
       <origin xyz="0 0 0.04" rpy="0 0 0"/>
     </collision>
+    <inertial>
+      <origin xyz="0 0 0.04" rpy="0 0 0"/>
+      <mass value="0.02"/>
+      <inertia ixx="0.000017" ixy="0" ixz="0" iyy="0.000011" iyz="0" izz="0.000007"/>
+    </inertial>
   </link>
   <!-- 左手指连接到底座 -->

Commit message: fix(description): stabilize Gazebo arm control
Lower position PID gains and drop the integral term to stop windup,
add joint dynamics damping, and raise base mass to 10 kg so the arm
stops oscillating/flying and holds its pose under gravity.

Co-Authored-By: deepseek <deepseek@users.noreply.github.com>

File: ros2_ws/src/my_robot_description/urdf/arm.xacro (robot description, xacro)
@@ -18,6 +18,6 @@
         <inertial>
             <origin xyz="0 0 0.05" rpy="0 0 0"/>
-            <mass value="5.0"/>
-            <inertia ixx="0.070833" ixy="0" ixz="0" iyy="0.070833" iyz="0" izz="0.133333"/>
+            <mass value="10.0"/>
+            <inertia ixx="0.141667" ixy="0" ixz="0" iyy="0.141667" iyz="0" izz="0.266667"/>
         </inertial>
     </link>
@@ -164,4 +164,5 @@
         <origin xyz="0 0 0.1" rpy="0 0 0"/>
         <axis xyz="0 0 1"/>
+        <dynamics damping="2.0"/>
         <limit lower="-3.14" upper="3.14" effort="1000.0" velocity="1.0"/>
     </joint>
@@ -172,4 +173,5 @@
         <origin xyz="0 0 0.5" rpy="0 0 0"/>
         <axis xyz="0 1 0"/>
+        <dynamics damping="2.0"/>
         <limit lower="0" upper="2.5" effort="1000.0" velocity="1.0"/>
     </joint>
@@ -180,4 +182,5 @@
         <origin xyz="0 0 0.6" rpy="0 0 0"/>
         <axis xyz="0 1 0"/>
+        <dynamics damping="2.0"/>
         <limit lower="0" upper="2.5" effort="1000.0" velocity="1.0"/>
     </joint>
@@ -188,4 +191,5 @@
         <origin xyz="0 0 0.1" rpy="0 0 0"/>
         <axis xyz="0 0 1"/>
+        <dynamics damping="2.0"/>
         <limit lower="-3.14" upper="3.14" effort="1000.0" velocity="1.0"/>
     </joint>
@@ -196,4 +200,5 @@
         <origin xyz="0 0 0.5" rpy="0 0 0"/>
         <axis xyz="0 1 0"/>
+        <dynamics damping="2.0"/>
         <limit lower="-1.57" upper="1.57" effort="1000.0" velocity="1.0"/>
     </joint>
@@ -204,4 +209,5 @@
         <origin xyz="0 0 0.05" rpy="0 0 0"/>
         <axis xyz="0 0 1"/>
+        <dynamics damping="2.0"/>
     </joint>
     <!-- hand_tool_joint: fixed -->

File: ros2_ws/src/my_robot_description/urdf/gripper.xacro (robot description, xacro)
@@ -70,4 +70,5 @@
     <origin xyz="-0.07 0 0.02" rpy="0 0 0"/>
     <axis xyz="1 0 0"/>
+    <dynamics damping="1.0"/>
     <limit effort="1000.0" velocity="1.0" lower="0.0" upper="0.06"/>
   </joint>

File: ros2_ws/src/my_robot_description/urdf/my_robot.gazebo.ros2_control.xacro (robot description, xacro)
@@ -5,6 +5,8 @@
     my_robot.ros2_control.xacro）：
     1) 硬件插件换成 gazebo_ros2_control/GazeboSystem，由 Gazebo 物理引擎驱动；
-    2) 每个关节的 position 命令接口通过 pos_kp/pos_ki/pos_kd 声明 PID 增益，
-       gazebo_ros2_control 会据此把位置误差换算成力矩作用到关节上（真实物理）；
+    2) 每个关节的 position 命令接口通过 pos_kp/pos_kd 声明 PID 增益，
+       gazebo_ros2_control 会据此把位置误差换算成力矩作用到关节上（真实物理）。
+       这里刻意去掉 pos_ki（积分项），避免 windup 导致臂发散；kd 加大 + URDF 里
+       的关节 dynamics damping 一起提供阻尼，防止振荡。
     3) 额外暴露 velocity 状态接口；
     4) <gazebo> 插件块 libgazebo_ros2_control.so 在模型加载时创建
@@ -16,7 +18,6 @@
     </hardware>
     <joint name="joint1">
-      <param name="pos_kp">100.0</param>
-      <param name="pos_ki">5.0</param>
-      <param name="pos_kd">1.0</param>
+      <param name="pos_kp">40.0</param>
+      <param name="pos_kd">10.0</param>
       <command_interface name="position"/>
       <state_interface name="position"/>
@@ -24,7 +25,6 @@
     </joint>
     <joint name="joint2">
-      <param name="pos_kp">100.0</param>
-      <param name="pos_ki">5.0</param>
-      <param name="pos_kd">1.0</param>
+      <param name="pos_kp">40.0</param>
+      <param name="pos_kd">10.0</param>
       <command_interface name="position"/>
       <state_interface name="position"/>
@@ -32,7 +32,6 @@
     </joint>
     <joint name="joint3">
-      <param name="pos_kp">100.0</param>
-      <param name="pos_ki">5.0</param>
-      <param name="pos_kd">1.0</param>
+      <param name="pos_kp">40.0</param>
+      <param name="pos_kd">10.0</param>
       <command_interface name="position"/>
       <state_interface name="position"/>
@@ -40,7 +39,6 @@
     </joint>
     <joint name="joint4">
-      <param name="pos_kp">100.0</param>
-      <param name="pos_ki">5.0</param>
-      <param name="pos_kd">1.0</param>
+      <param name="pos_kp">40.0</param>
+      <param name="pos_kd">10.0</param>
       <command_interface name="position"/>
       <state_interface name="position"/>
@@ -48,7 +46,6 @@
     </joint>
     <joint name="joint5">
-      <param name="pos_kp">100.0</param>
-      <param name="pos_ki">5.0</param>
-      <param name="pos_kd">1.0</param>
+      <param name="pos_kp">40.0</param>
+      <param name="pos_kd">10.0</param>
       <command_interface name="position"/>
       <state_interface name="position"/>
@@ -56,7 +53,6 @@
     </joint>
     <joint name="joint6">
-      <param name="pos_kp">100.0</param>
-      <param name="pos_ki">5.0</param>
-      <param name="pos_kd">1.0</param>
+      <param name="pos_kp">40.0</param>
+      <param name="pos_kd">10.0</param>
       <command_interface name="position"/>
       <state_interface name="position"/>
@@ -64,7 +60,6 @@
     </joint>
     <joint name="gripper_left_finger_joint">
-      <param name="pos_kp">50.0</param>
-      <param name="pos_ki">1.0</param>
-      <param name="pos_kd">0.5</param>
+      <param name="pos_kp">20.0</param>
+      <param name="pos_kd">2.0</param>
       <command_interface name="position"/>
       <state_interface name="position"/>

Commit message: fix(description): increase link masses and retune PID
The arm links were unrealistically light (0.1-0.5 kg), giving tiny
inertia that made the sim numerically unstable (fly-away or collapse).
Raise link masses to realistic values, and retune the position PID
(kp 80, kd 15, no integral) for the heavier arm.

Co-Authored-By: deepseek <deepseek@users.noreply.github.com>

File: ros2_ws/src/my_robot_description/urdf/arm.xacro (robot description, xacro)
@@ -39,6 +39,6 @@
         <inertial>
             <origin xyz="0 0 0.25" rpy="0 0 0"/>
-            <mass value="0.5"/>
-            <inertia ixx="0.011667" ixy="0" ixz="0" iyy="0.011667" iyz="0" izz="0.0025"/>
+            <mass value="1.0"/>
+            <inertia ixx="0.023333" ixy="0" ixz="0" iyy="0.023333" iyz="0" izz="0.005"/>
         </inertial>
     </link>
@@ -61,6 +61,6 @@
         <inertial>
             <origin xyz="0 0 0.3" rpy="0 0 0"/>
-            <mass value="0.3"/>
-            <inertia ixx="0.009188" ixy="0" ixz="0" iyy="0.009188" iyz="0" izz="0.000375"/>
+            <mass value="1.0"/>
+            <inertia ixx="0.030625" ixy="0" ixz="0" iyy="0.030625" iyz="0" izz="0.00125"/>
         </inertial>
     </link>
@@ -82,6 +82,6 @@
         <inertial>
             <origin xyz="0 0 0.05" rpy="0 0 0"/>
-            <mass value="0.1"/>
-            <inertia ixx="0.000146" ixy="0" ixz="0" iyy="0.000146" iyz="0" izz="0.000125"/>
+            <mass value="0.5"/>
+            <inertia ixx="0.000729" ixy="0" ixz="0" iyy="0.000729" iyz="0" izz="0.000625"/>
         </inertial>
     </link>
@@ -104,6 +104,6 @@
         <inertial>
             <origin xyz="0 0 0.25" rpy="0 0 0"/>
-            <mass value="0.25"/>
-            <inertia ixx="0.005365" ixy="0" ixz="0" iyy="0.005365" iyz="0" izz="0.000313"/>
+            <mass value="0.8"/>
+            <inertia ixx="0.017167" ixy="0" ixz="0" iyy="0.017167" iyz="0" izz="0.001"/>
         </inertial>
     </link>
@@ -125,6 +125,6 @@
         <inertial>
             <origin xyz="0 0 0.025" rpy="0 0 0"/>
-            <mass value="0.1"/>
-            <inertia ixx="0.000104" ixy="0" ixz="0" iyy="0.000104" iyz="0" izz="0.000167"/>
+            <mass value="0.3"/>
+            <inertia ixx="0.000313" ixy="0" ixz="0" iyy="0.000313" iyz="0" izz="0.0005"/>
         </inertial>
     </link>
@@ -146,6 +146,6 @@
         <inertial>
             <origin xyz="0 0 0.01" rpy="0 0 0"/>
-            <mass value="0.05"/>
-            <inertia ixx="0.000043" ixy="0" ixz="0" iyy="0.000043" iyz="0" izz="0.000083"/>
+            <mass value="0.2"/>
+            <inertia ixx="0.000173" ixy="0" ixz="0" iyy="0.000173" iyz="0" izz="0.000333"/>
         </inertial>
     </link>
@@ -154,6 +154,6 @@
         <inertial>
             <origin xyz="0 0 0" rpy="0 0 0"/>
-            <mass value="0.01"/>
-            <inertia ixx="0.000001" ixy="0" ixz="0" iyy="0.000001" iyz="0" izz="0.000001"/>
+            <mass value="0.05"/>
+            <inertia ixx="0.000005" ixy="0" ixz="0" iyy="0.000005" iyz="0" izz="0.000005"/>
         </inertial>
     </link>

File: ros2_ws/src/my_robot_description/urdf/gripper.xacro (robot description, xacro)
@@ -18,6 +18,6 @@
     <inertial>
       <origin xyz="0 0 0.01" rpy="0 0 0"/>
-      <mass value="0.05"/>
-      <inertia ixx="0.000017" ixy="0" ixz="0" iyy="0.000168" iyz="0" izz="0.000182"/>
+      <mass value="0.2"/>
+      <inertia ixx="0.000067" ixy="0" ixz="0" iyy="0.000673" iyz="0" izz="0.000727"/>
     </inertial>
   </link>
@@ -39,6 +39,6 @@
     <inertial>
       <origin xyz="0 0 0.04" rpy="0 0 0"/>
-      <mass value="0.02"/>
-      <inertia ixx="0.000017" ixy="0" ixz="0" iyy="0.000011" iyz="0" izz="0.000007"/>
+      <mass value="0.08"/>
+      <inertia ixx="0.000067" ixy="0" ixz="0" iyy="0.000045" iyz="0" izz="0.000027"/>
     </inertial>
   </link>
@@ -60,6 +60,6 @@
     <inertial>
       <origin xyz="0 0 0.04" rpy="0 0 0"/>
-      <mass value="0.02"/>
-      <inertia ixx="0.000017" ixy="0" ixz="0" iyy="0.000011" iyz="0" izz="0.000007"/>
+      <mass value="0.08"/>
+      <inertia ixx="0.000067" ixy="0" ixz="0" iyy="0.000045" iyz="0" izz="0.000027"/>
     </inertial>
   </link>

File: ros2_ws/src/my_robot_description/urdf/my_robot.gazebo.ros2_control.xacro (robot description, xacro)
@@ -18,6 +18,6 @@
     </hardware>
     <joint name="joint1">
-      <param name="pos_kp">40.0</param>
-      <param name="pos_kd">10.0</param>
+      <param name="pos_kp">80.0</param>
+      <param name="pos_kd">15.0</param>
       <command_interface name="position"/>
       <state_interface name="position"/>
@@ -25,6 +25,6 @@
     </joint>
     <joint name="joint2">
-      <param name="pos_kp">40.0</param>
-      <param name="pos_kd">10.0</param>
+      <param name="pos_kp">80.0</param>
+      <param name="pos_kd">15.0</param>
       <command_interface name="position"/>
       <state_interface name="position"/>
@@ -32,6 +32,6 @@
     </joint>
     <joint name="joint3">
-      <param name="pos_kp">40.0</param>
-      <param name="pos_kd">10.0</param>
+      <param name="pos_kp">80.0</param>
+      <param name="pos_kd">15.0</param>
       <command_interface name="position"/>
       <state_interface name="position"/>
@@ -39,6 +39,6 @@
     </joint>
     <joint name="joint4">
-      <param name="pos_kp">40.0</param>
-      <param name="pos_kd">10.0</param>
+      <param name="pos_kp">80.0</param>
+      <param name="pos_kd">15.0</param>
       <command_interface name="position"/>
       <state_interface name="position"/>
@@ -46,6 +46,6 @@
     </joint>
     <joint name="joint5">
-      <param name="pos_kp">40.0</param>
-      <param name="pos_kd">10.0</param>
+      <param name="pos_kp">80.0</param>
+      <param name="pos_kd">15.0</param>
       <command_interface name="position"/>
       <state_interface name="position"/>
@@ -53,6 +53,6 @@
     </joint>
     <joint name="joint6">
-      <param name="pos_kp">40.0</param>
-      <param name="pos_kd">10.0</param>
+      <param name="pos_kp">80.0</param>
+      <param name="pos_kd">15.0</param>
       <command_interface name="position"/>
       <state_interface name="position"/>
@@ -60,6 +60,6 @@
     </joint>
     <joint name="gripper_left_finger_joint">
-      <param name="pos_kp">20.0</param>
-      <param name="pos_kd">2.0</param>
+      <param name="pos_kp">30.0</param>
+      <param name="pos_kd">3.0</param>
       <command_interface name="position"/>
       <state_interface name="position"/>

Commit message: fix(gazebo): revert the disable_collide block, leave gaps between links
The <gazebo><joint><disable_collide> form broke model spawning
outright:

  Error Code 4 Msg: Required attribute[type] in element[joint] is not
  specified in SDF.

Gazebo reads the spawned URDF through sdf::readString(), which hands
the robot-level <gazebo> children to the SDF parser; a <joint> there
without a type attribute makes the whole model fail to load. Reverted.

Instead, remove the degenerate contacts geometrically: every arm link's
collision box used to end exactly where the next one began (and with
fully overlapping x/y footprints), and base_link's bottom face sat
exactly on the z=0 ground plane. Zero-penetration, face-to-face
contacts are degenerate input for ODE's constraint solver. Each box is
now 1 cm shorter along the joint axis, so neighbouring links keep a
>=1.5 cm gap.

Also write the expanded URDF to /tmp and dump Gazebo's real per-link
poses plus the URDF->SDF conversion result, so the model state can be
inspected without a screenshot.

Co-Authored-By: deepseek <deepseek@anthropic.com>

File: ros2_ws/src/my_robot_description/urdf/arm.xacro (robot description, xacro)
@@ -12,7 +12,7 @@
         <collision>
             <geometry>
-                <box size="0.4 0.4 0.1"/>
-            </geometry>
-            <origin xyz="0 0 0.05" rpy="0 0 0"/>
+                <box size="0.4 0.4 0.09"/>
+            </geometry>
+            <origin xyz="0 0 0.045" rpy="0 0 0"/>
         </collision>
         <inertial>
@@ -33,5 +33,5 @@
         <collision>
             <geometry>
-                <box size="0.2 0.2 0.5"/>
+                <box size="0.2 0.2 0.48"/>
             </geometry>
             <origin xyz="0 0 0.25" rpy="0 0 0"/>
@@ -55,5 +55,5 @@
         <collision>
             <geometry>
-                <box size="0.1 0.1 0.6"/>
+                <box size="0.1 0.1 0.58"/>
             </geometry>
             <origin xyz="0 0 0.3" rpy="0 0 0"/>
@@ -76,5 +76,5 @@
         <collision>
             <geometry>
-                <box size="0.1 0.1 0.1"/>
+                <box size="0.1 0.1 0.08"/>
             </geometry>
             <origin xyz="0 0 0.05" rpy="0 0 0"/>
@@ -98,5 +98,5 @@
         <collision>
             <geometry>
-                <box size="0.1 0.1 0.5"/>
+                <box size="0.1 0.1 0.48"/>
             </geometry>
             <origin xyz="0 0 0.25" rpy="0 0 0"/>
@@ -119,5 +119,5 @@
         <collision>
             <geometry>
-                <box size="0.1 0.1 0.05"/>
+                <box size="0.1 0.1 0.03"/>
             </geometry>
             <origin xyz="0 0 0.025" rpy="0 0 0"/>
@@ -140,5 +140,5 @@
         <collision>
             <geometry>
-                <box size="0.1 0.1 0.02"/>
+                <box size="0.1 0.1 0.01"/>
             </geometry>
             <origin xyz="0 0 0.01" rpy="0 0 0"/>

File: ros2_ws/src/my_robot_description/urdf/my_robot.gazebo.ros2_control.xacro (robot description, xacro)
@@ -75,42 +75,10 @@
     </plugin>
   </gazebo>
-  <!-- 关闭相邻连杆之间的碰撞。
-       本 URDF 里每一段的碰撞盒都"正好贴着"下一段（面面共面，X/Y 完全重叠），
-       这种零穿透的退化接触会让 ODE 的约束求解器解出 NaN：
-       关节 velocity/effort 变成 NaN，连杆位姿变成 NaN，
-       Gazebo 渲染时 NaN 位姿的连杆直接不显示 —— 表现就是"只剩底座，机械臂不见了"。
-       机器人自身的相邻连杆本来就不该互相碰撞，关掉同时也避免
-       碰撞求解器跟关节 PID 抢力矩（机械臂会抖、会飞）。 -->
-  <gazebo>
-    <joint name="joint1">
-      <parent>base_link</parent>
-      <child>shoulder_link</child>
-      <disable_collide>true</disable_collide>
-    </joint>
-    <joint name="joint2">
-      <parent>shoulder_link</parent>
-      <child>arm_link</child>
-      <disable_collide>true</disable_collide>
-    </joint>
-    <joint name="joint3">
-      <parent>arm_link</parent>
-      <child>elbow_link</child>
-      <disable_collide>true</disable_collide>
-    </joint>
-    <joint name="joint4">
-      <parent>elbow_link</parent>
-      <child>forearm_link</child>
-      <disable_collide>true</disable_collide>
-    </joint>
-    <joint name="joint5">
-      <parent>forearm_link</parent>
-      <child>wrist_link</child>
-      <disable_collide>true</disable_collide>
-    </joint>
-    <joint name="joint6">
-      <parent>wrist_link</parent>
-      <child>hand_link</child>
-      <disable_collide>true</disable_collide>
-    </joint>
-  </gazebo>
+  <!--
+    注意：不要在这里加 <gazebo><joint>...<disable_collide> 的写法。
+    Gazebo 把 URDF 读进来时会把它当成真正的 SDF <joint> 处理，而
+    disable_collide 那种写法没有 type 属性，结果是整个模型解析失败：
+      Error Code 4 Msg: Required attribute[type] in element[joint] is not specified in SDF.
+    相邻连杆的碰撞改用 arm.xacro 里的碰撞盒留缝（每段比原来短 1cm）来避免。
+  -->
 </robot>
