Commit message: fix(description): drop mimic and velocity state to fix NaN
Gazebo produces NaN for the prismatic mimic finger joint, which corrupts
the gripper TF. Make the right finger a fixed joint and drop the velocity
state interface (unused by the position controller) so /joint_states is
clean.

Co-Authored-By: deepseek <deepseek@users.noreply.github.com>

File: ros2_ws/src/my_robot_description/urdf/gripper.xacro (robot description, xacro)
@@ -73,12 +73,9 @@
     <limit effort="1000.0" velocity="1.0" lower="0.0" upper="0.06"/>
   </joint>
-  <!-- 右手指连接到底座 -->
-  <joint name="gripper_right_finger_joint" type="prismatic">
+  <!-- 右手指固定连接到底座（Gazebo 对 mimic 联动不稳定，改为固定） -->
+  <joint name="gripper_right_finger_joint" type="fixed">
     <parent link="gripper_base_link"/>
     <child link="gripper_right_finger_link"/>
     <origin xyz="0.07 0 0.02" rpy="0 0 0"/>
-    <axis xyz="1 0 0"/>
-    <mimic joint="gripper_left_finger_joint" multiplier="-1.0"/>
-    <limit effort="1000.0" velocity="1.0" lower="-0.06" upper="0.0"/>
   </joint>
 </robot>

File: ros2_ws/src/my_robot_description/urdf/my_robot.gazebo.ros2_control.xacro (robot description, xacro)
@@ -22,5 +22,4 @@
       <command_interface name="position"/>
       <state_interface name="position"/>
-      <state_interface name="velocity"/>
     </joint>
     <joint name="joint2">
@@ -29,5 +28,4 @@
       <command_interface name="position"/>
       <state_interface name="position"/>
-      <state_interface name="velocity"/>
     </joint>
     <joint name="joint3">
@@ -36,5 +34,4 @@
       <command_interface name="position"/>
       <state_interface name="position"/>
-      <state_interface name="velocity"/>
     </joint>
     <joint name="joint4">
@@ -43,5 +40,4 @@
       <command_interface name="position"/>
       <state_interface name="position"/>
-      <state_interface name="velocity"/>
     </joint>
     <joint name="joint5">
@@ -50,5 +46,4 @@
       <command_interface name="position"/>
       <state_interface name="position"/>
-      <state_interface name="velocity"/>
     </joint>
     <joint name="joint6">
@@ -57,5 +52,4 @@
       <command_interface name="position"/>
       <state_interface name="position"/>
-      <state_interface name="velocity"/>
     </joint>
     <joint name="gripper_left_finger_joint">
@@ -64,5 +58,4 @@
       <command_interface name="position"/>
       <state_interface name="position"/>
-      <state_interface name="velocity"/>
     </joint>
   </ros2_control>

Commit message: fix(description): drop gripper control to resolve prismatic NaN
The prismatic finger joint returns NaN position in gazebo_ros2_control
regardless of mimic/velocity settings. Make the gripper a fixed assembly
and remove it from ros2_control and the controller spawner, so the 6-DOF
arm is fully controllable.

Co-Authored-By: deepseek <deepseek@users.noreply.github.com>

File: ros2_ws/src/my_robot_description/urdf/gripper.xacro (robot description, xacro)
@@ -64,12 +64,9 @@
     </inertial>
   </link>
-  <!-- 左手指连接到底座 -->
-  <joint name="gripper_left_finger_joint" type="prismatic">
+  <!-- 左手指固定连接到底座（Gazebo 下 prismatic 关节有 NaN 问题，先改为固定） -->
+  <joint name="gripper_left_finger_joint" type="fixed">
     <parent link="gripper_base_link"/>
     <child link="gripper_left_finger_link"/>
     <origin xyz="-0.07 0 0.02" rpy="0 0 0"/>
-    <axis xyz="1 0 0"/>
-    <dynamics damping="1.0"/>
-    <limit effort="1000.0" velocity="1.0" lower="0.0" upper="0.06"/>
   </joint>
   <!-- 右手指固定连接到底座（Gazebo 对 mimic 联动不稳定，改为固定） -->

File: ros2_ws/src/my_robot_description/urdf/my_robot.gazebo.ros2_control.xacro (robot description, xacro)
@@ -53,10 +53,4 @@
       <state_interface name="position"/>
     </joint>
-    <joint name="gripper_left_finger_joint">
-      <param name="pos_kp">30.0</param>
-      <param name="pos_kd">3.0</param>
-      <command_interface name="position"/>
-      <state_interface name="position"/>
-    </joint>
   </ros2_control>
   <!-- Gazebo 加载该插件，创建 controller_manager 并读取控制器参数 -->

Commit message: feat(gazebo): re-enable gripper control with prismatic + mimic joints
Restore the tutorial's original gripper design so the fingers can open and
close under Gazebo physics again:

- gripper.xacro: change both finger joints from fixed back to prismatic.
  The left finger is the controlled joint (axis +x, 0..0.06); the right
  finger is a mimic joint (multiplier -1.0) that follows it, so one command
  drives both fingers symmetrically.
- my_robot.gazebo.ros2_control.xacro: declare gripper_left_finger_joint in
  the GazeboSystem hardware interface (position command + position/velocity
  state interfaces, initial_value 0).
- ros2_controllers_gazebo.yaml: add gripper_controller (JointTrajectoryController
  over gripper_left_finger_joint).
- gazebo.launch.py: spawn gripper_controller alongside the arm controllers.

The earlier "prismatic NaN" was a symptom of the then-unstable model (ODE step
size + PID torque thread race), which the visibility fixes have since resolved,
so the joint can be restored without re-architecting the gripper.

Co-Authored-By: deepseek <deepseek@users.noreply.github.com>

File: ros2_ws/src/my_robot_description/urdf/gripper.xacro (robot description, xacro)
@@ -64,15 +64,24 @@
     </inertial>
   </link>
-  <!-- 左手指固定连接到底座（Gazebo 下 prismatic 关节有 NaN 问题，先改为固定） -->
-  <joint name="gripper_left_finger_joint" type="fixed">
+  <!-- 左手指连接到底座（prismatic，axis=+x，0=张开 0.06=闭合）。
+       damping 给一点阻尼，避免这节低质量滑动关节在位置控制下抖动。 -->
+  <joint name="gripper_left_finger_joint" type="prismatic">
     <parent link="gripper_base_link"/>
     <child link="gripper_left_finger_link"/>
     <origin xyz="-0.07 0 0.02" rpy="0 0 0"/>
+    <axis xyz="1 0 0"/>
+    <dynamics damping="1.0"/>
+    <limit effort="1000.0" velocity="1.0" lower="0.0" upper="0.06"/>
   </joint>
-  <!-- 右手指固定连接到底座（Gazebo 对 mimic 联动不稳定，改为固定） -->
-  <joint name="gripper_right_finger_joint" type="fixed">
+  <!-- 右手指连接到底座：mimic 联动左手指，multiplier=-1.0 表示反向，
+       左手指动多少它就反向动多少，两指对向开合。右手指只做从动，
+       不放进 ros2_control，由 Gazebo 物理引擎按 mimic 关系自动跟随。 -->
+  <joint name="gripper_right_finger_joint" type="prismatic">
     <parent link="gripper_base_link"/>
     <child link="gripper_right_finger_link"/>
     <origin xyz="0.07 0 0.02" rpy="0 0 0"/>
+    <axis xyz="1 0 0"/>
+    <mimic joint="gripper_left_finger_joint" multiplier="-1.0"/>
+    <limit effort="1000.0" velocity="1.0" lower="-0.06" upper="0.0"/>
   </joint>
 </robot>

File: ros2_ws/src/my_robot_description/urdf/my_robot.gazebo.ros2_control.xacro (robot description, xacro)
@@ -96,4 +96,13 @@
       <state_interface name="velocity"/>
     </joint>
+    <joint name="gripper_left_finger_joint">
+      <command_interface name="position"/>
+      <state_interface name="position">
+        <param name="initial_value">0.0</param>
+      </state_interface>
+      <!-- 速度状态接口：不声明的话 joint_state_broadcaster 会往
+           /joint_states 里发 NaN 速度（没有可用的状态接口） -->
+      <state_interface name="velocity"/>
+    </joint>
   </ros2_control>
   <!-- Gazebo 加载该插件，创建 controller_manager 并读取控制器参数。
